Commit message: stack_up.py added

File: robots/universal_robot/ur_description/urdf/inc/ur5e_macro.xacro (robot description, xacro)
@@ -40,4 +40,26 @@
       safety_k_position="${safety_k_position}"
     />
+    <link name="ur5e_table_link">
+      <visual>
+        <origin xyz="0 0 0.71" rpy="0 0 -1.57" />
+        <geometry>
+          <mesh filename="package://ur5e_robotiq_description/meshes/UR5e_table.stl"/>
+        </geometry>
+        <material name="light_grey">
+          <color rgba="0.75 0.75 0.75 1"/>
+        </material>
+      </visual>
+      <collision>
+        <origin xyz="0 0 0" rpy="0 0 0"/>
+        <geometry>
+          <mesh filename="package://ur5e_robotiq_description/meshes/UR5e_table.stl"/>
+        </geometry>
+      </collision>
+    </link>
+    <joint name="ur5e_table_joint" type="fixed">
+      <parent link="ur5e_table_link"/>
+      <child link="${prefix}base_link"/>
+      <origin xyz="0 0 0.71" rpy="0 0 0"/>
+     </joint>
   </xacro:macro>
 </robot>

File: ur5e_robotiq_moveit/config/gazebo_ur5e_robot.urdf (robot description, URDF)
Before this commit: robot ur5e_robot, 21 links, 20 joints
Links:
- added link ur5e_table_link, mass 100.0; collision mesh filename=package://ur5e_robotiq_description/meshes/UR5e_table.stl; visual mesh filename=package://ur5e_robotiq_description/meshes/UR5e_table.stl
Joints:
- added joint ur5e_table_joint: type fixed, parent ur5e_table_link, child base_link, origin xyz=0 0 0.71 rpy=0 0 0
- joint world_joint: child base_link -> ur5e_table_link
